File: BeeBoardHardware.kicad_sch (KiCad schematic)
At the start: 46 parts, among them J2 USB_C_Receptacle_USB2.0_16P, J3 Conn_01x02, J4 Conn_01x11, Q1 AO3413, SW2 SW_Push, U1 MCP16311x-xMNY, U2 BQ24074RGT, U3 USBLC6-2SC6, U4 LC709203FQH-01TWG, U5 STM6600DQ25DM6F

Commit message: routing headers next
Parts:
- removed H3, H4: MountingHole, MountingHole:MountingHole_2.1mm, symbol Mechanical:MountingHole
- J4: Digikey Link (none) -> https://www.digikey.com/en/products/detail/adam-tech/PH1-11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; Manufacturer Product Number (none) -> PH1-11-UA
- U1: value MCP16311x-xMNY -> MCP16311T-E/MNY; Digikey Link (none) -> https://www.digikey.com/en/products/detail/microchip-techno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; Manufacturer Product Number (none) -> MCP16311T-E/MNY
- U2: value BQ24074RGT -> BQ24074RGTT; Digikey Link (none) -> https://www.digikey.com/en/products/detail/texas-instrument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; Manufacturer Product Number (none) -> BQ24074RGTT
- U4: Digikey Link (none) -> https://www.digikey.com/en/products/detail/onsemi/LC709203F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; Manufacturer Product Number (none) -> LC709203FQH-01TWG
- U5: Digikey Link (none) -> https://www.digikey.com/en/products/detail/stmicroelectroni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; Manufacturer Product Number (none) -> STM6600DQ25DM6F
